Commit message: Simulation Done

File: src/roguetwo_description/urdf/em_3905.urdf.xacro (robot description, xacro)
@@ -358,5 +358,102 @@
   <xacro:rear_wheel lr_prefix="right" fr_prefix="rear"
                     lr_reflect="-1" fr_reflect="-1"/>
-  <link name="camera_stereo_left">
+  <xacro:property name="height1" value="0.05" />
+  <xacro:property name="width" value="0.05" />
+  <joint name="fixed" type="fixed">
+    <parent link="chassis"/>
+    <child link="sensor"/>
+  </joint>
+ <!-- Base Link -->
+  <link name="sensor">
+    <collision>
+      <origin xyz="0 0 ${height1/2}" rpy="0 0 0"/>
+      <geometry>
+        <box size="${width} ${width} ${height1}"/>
+      </geometry>
+    </collision>
+    <visual>
+      <origin xyz="0 0 ${height1/2}" rpy="0 0 0"/>
+      <geometry>
+        <box size="${width} ${width} ${height1}"/>
+      </geometry>
+      <material name="orange"/>
+    </visual>
+    <inertial>
+      <origin xyz="0 0 0.1" rpy="0 0 0"/>
+      <mass value="1"/>
+      <inertia
+        ixx="1.0" ixy="0.0" ixz="0.0"
+        iyy="1.0" iyz="0.0"
+        izz="1.0"/>
+    </inertial>
+  </link>
+  <joint name="stereo_joint" type="fixed">
+    <axis xyz="0 1 0" />
+    <origin xyz=".1 .0 0.1" rpy="0 0 0"/>
+    <parent link="base_link"/>
+    <child link="sensor"/>
+  </joint>
+  <material name="orange">
+    <color rgba="${255/255} ${108/255} ${10/255} 1.0"/>
+  </material>
+ <gazebo reference="sensor">
+    <material>Gazebo/Orange</material>
+  </gazebo>
+  <gazebo reference="sensor">
+    <sensor type="multicamera" name="stereo_camera">
+      <update_rate>30.0</update_rate>
+      <camera name="left">
+        <horizontal_fov>1.3962634</horizontal_fov>
+        <image>
+          <width>640</width>
+          <height>480</height>
+          <format>R8G8B8</format>
+        </image>
+        <clip>
+          <near>0.02</near>
+          <far>300</far>
+        </clip>
+        <noise>
+          <type>gaussian</type>
+          <mean>0.0</mean>
+          <stddev>0.007</stddev>
+        </noise>
+      </camera>
+      <camera name="right">
+        <pose>0 -0.07 0 0 0 0</pose>
+        <horizontal_fov>1.3962634</horizontal_fov>
+        <image>
+          <width>640</width>
+          <height>480</height>
+          <format>R8G8B8</format>
+        </image>
+        <clip>
+          <near>0.02</near>
+          <far>300</far>
+        </clip>
+        <noise>
+          <type>gaussian</type>
+          <mean>0.0</mean>
+          <stddev>0.007</stddev>
+        </noise>
+      </camera>
+      <plugin name="stereo_camera_controller" filename="libgazebo_ros_multicamera.so">
+        <alwaysOn>true</alwaysOn>
+        <updateRate>0.0</updateRate>
+        <cameraName>stereo/camera</cameraName>
+        <imageTopicName>image_raw</imageTopicName>
+        <cameraInfoTopicName>camera_info</cameraInfoTopicName>
+        <frameName>left_camera_optical_frame</frameName>
+        <!--<rightFrameName>right_camera_optical_frame</rightFrameName>-->
+        <hackBaseline>0.07</hackBaseline>
+        <distortionK1>0.0</distortionK1>
+        <distortionK2>0.0</distortionK2>
+        <distortionK3>0.0</distortionK3>
+        <distortionT1>0.0</distortionT1>
+        <distortionT2>0.0</distortionT2>
+      </plugin>
+    </sensor>
+  </gazebo>
+<!--   <link name="camera_stereo_left">
     <collision>
       <origin xyz="0 0 0" rpy="0 0 0"/>
@@ -535,4 +632,5 @@
     </sensor>
   </gazebo>
+ -->
 <!--   <xacro:property name="height1" value="0.2" />
   <xacro:property name="width" value="0.2" /> -->
@@ -609,4 +707,76 @@
     <child link="imu"/>
   </joint>
+  <xacro:property name="height_sonar" value="0.05" />
+  <xacro:property name="width_sonar" value="0.05" />
+  <xacro:property name="name" value="sonar" />
+  <xacro:property name="ros_topic" value="/sonar_distance" />
+  <xacro:property name="update_rate" value="10" />
+  <xacro:property name="min_range" value="0.02" />
+  <xacro:property name="max_range" value="5.0" />
+  <xacro:property name="field_of_view" value="15" />
+  <xacro:property name="ray_count" value="8" />
+  <!-- Base Link -->
+  <link name="${name}_link">
+      <inertial>
+        <mass value="0.001" />
+        <origin xyz="0 0 0" rpy="0 0 0" />
+        <inertia ixx="0.000000017" ixy="0" ixz="0" iyy="0.000000017" iyz="0" izz="0.000000017" />
+      </inertial>
+        <visual>
+          <origin xyz="0 0 ${height_sonar/2}" rpy="0 0 0"/>
+          <geometry>
+            <box size="${width_sonar} ${width_sonar} ${height_sonar}"/>
+          </geometry>
+          <material name="orange"/>
+        </visual>
+      <collision>
+        <origin xyz="0 0 0" rpy="0 0 0" />
+        <geometry>
+          <box size="0.01 0.01 0.01" />
+        </geometry>
+      </collision>
+  </link>
+  <joint name="${name}_joint" type="fixed">
+    <axis xyz="0 1 0" />
+    <origin xyz=".15 .0 0.0" rpy="0 0 0"/>
+    <parent link="chassis"/>
+    <child link="${name}_link"/>
+  </joint>
+    <gazebo reference="${name}_link">
+      <sensor type="ray" name="${name}">
+        <always_on>true</always_on>
+        <update_rate>${update_rate}</update_rate>
+        <pose>0 0 0 0 0 0</pose>
+        <visualize>false</visualize>
+        <ray>
+          <scan>
+            <horizontal>
+              <samples>${ray_count}</samples>
+              <resolution>1</resolution>
+              <min_angle>-${field_of_view/2}</min_angle>
+              <max_angle> ${field_of_view/2}</max_angle>
+            </horizontal>
+            <vertical>
+              <samples>${ray_count}</samples>
+              <resolution>1</resolution>
+              <min_angle>-${field_of_view/2}</min_angle>
+              <max_angle> ${field_of_view/2}</max_angle>
+            </vertical>
+          </scan>
+          <range>
+            <min>${min_range}</min>
+            <max>${max_range}</max>
+            <resolution>0.01</resolution>
+          </range>
+        </ray>
+        <plugin name="gazebo_ros_${name}_controller" filename="libhector_gazebo_ros_sonar.so">
+          <gaussianNoise>0.005</gaussianNoise>
+          <topicName>${ros_topic}</topicName>
+          <bodyName>sonar</bodyName>
+          <serviceName>sonar_service</serviceName>
+          <frameId>${name}_link</frameId>
+        </plugin>
+      </sensor>
+    </gazebo>
   <gazebo>
     <plugin name="imu_plugin" filename="libgazebo_ros_imu.so">
@@ -615,5 +785,5 @@
       <topicName>imu</topicName>
       <serviceName>imu_service</serviceName>
-      <gaussianNoise>0.0</gaussianNoise>
+      <gaussianNoise>0.005</gaussianNoise>
       <updateRate>20.0</updateRate>
     </plugin>

Commit message: Sonars Working Correctly

File: src/roguetwo_description/urdf/em_3905.urdf.xacro (robot description, xacro)
@@ -709,13 +709,19 @@
   <xacro:property name="height_sonar" value="0.05" />
   <xacro:property name="width_sonar" value="0.05" />
-  <xacro:property name="name" value="sonar" />
-  <xacro:property name="ros_topic" value="/sonar_distance" />
+  <xacro:property name="name1" value="sonar1" />
+  <xacro:property name="name2" value="sonar2" />
+  <xacro:property name="name3" value="sonar3" />
+  <xacro:property name="name4" value="sonar4" />
+  <xacro:property name="ros_topic1" value="/sonar_front_distance" />
+  <xacro:property name="ros_topic2" value="/sonar_left_distance" />
+  <xacro:property name="ros_topic3" value="/sonar_right_distance" />
+  <xacro:property name="ros_topic4" value="/sonar_back_distance" />
   <xacro:property name="update_rate" value="10" />
   <xacro:property name="min_range" value="0.02" />
-  <xacro:property name="max_range" value="5.0" />
-  <xacro:property name="field_of_view" value="15" />
-  <xacro:property name="ray_count" value="8" />
+  <xacro:property name="max_range" value="4.5" />
+  <xacro:property name="field_of_view" value="1" />
+  <xacro:property name="ray_count" value="2" />
   <!-- Base Link -->
-  <link name="${name}_link">
+  <link name="${name1}_link">
       <inertial>
         <mass value="0.001" />
@@ -737,16 +743,16 @@
       </collision>
   </link>
-  <joint name="${name}_joint" type="fixed">
+  <joint name="${name1}_joint" type="fixed">
     <axis xyz="0 1 0" />
-    <origin xyz=".15 .0 0.0" rpy="0 0 0"/>
+    <origin xyz=".25 0 0.15" rpy="0 -0.7 0"/>
     <parent link="chassis"/>
-    <child link="${name}_link"/>
-  </joint>
-    <gazebo reference="${name}_link">
-      <sensor type="ray" name="${name}">
+    <child link="${name1}_link"/>
+  </joint>
+    <gazebo reference="${name1}_link">
+      <sensor type="ray" name="${name1}">
         <always_on>true</always_on>
         <update_rate>${update_rate}</update_rate>
         <pose>0 0 0 0 0 0</pose>
-        <visualize>false</visualize>
+        <visualize>true</visualize>
         <ray>
           <scan>
@@ -770,10 +776,195 @@
           </range>
         </ray>
-        <plugin name="gazebo_ros_${name}_controller" filename="libhector_gazebo_ros_sonar.so">
+        <plugin name="gazebo_ros_${name1}_controller" filename="libhector_gazebo_ros_sonar.so">
           <gaussianNoise>0.005</gaussianNoise>
-          <topicName>${ros_topic}</topicName>
+          <topicName>${ros_topic1}</topicName>
+          <frameId>${name1}_link</frameId>
+        </plugin>
+      </sensor>
+    </gazebo>
+  <!-- Base Link -->
+  <link name="${name2}_link">
+      <inertial>
+        <mass value="0.001" />
+        <origin xyz="0 0 0" rpy="0 0 0" />
+        <inertia ixx="0.000000017" ixy="0" ixz="0" iyy="0.000000017" iyz="0" izz="0.000000017" />
+      </inertial>
+        <visual>
+          <origin xyz="0 0 ${height_sonar/2}" rpy="0 0 0"/>
+          <geometry>
+            <box size="${width_sonar} ${width_sonar} ${height_sonar}"/>
+          </geometry>
+          <material name="orange"/>
+        </visual>
+      <collision>
+        <origin xyz="0 0 0" rpy="0 0 0" />
+        <geometry>
+          <box size="0.01 0.01 0.01" />
+        </geometry>
+      </collision>
+  </link>
+  <joint name="${name2}_joint" type="fixed">
+    <axis xyz="0 1 0" />
+    <origin xyz=".0 .25 0.15" rpy="0 -0.60 1.5"/>
+    <parent link="chassis"/>
+    <child link="${name2}_link"/>
+  </joint>
+    <gazebo reference="${name2}_link">
+      <sensor type="ray" name="${name2}">
+        <always_on>true</always_on>
+        <update_rate>${update_rate}</update_rate>
+        <pose>0 0 0 0 0 0</pose>
+        <visualize>true</visualize>
+        <ray>
+          <scan>
+            <horizontal>
+              <samples>${ray_count}</samples>
+              <resolution>1</resolution>
+              <min_angle>-${field_of_view/2}</min_angle>
+              <max_angle> ${field_of_view/2}</max_angle>
+            </horizontal>
+            <vertical>
+              <samples>${ray_count}</samples>
+              <resolution>1</resolution>
+              <min_angle>-${field_of_view/2}</min_angle>
+              <max_angle> ${field_of_view/2}</max_angle>
+            </vertical>
+          </scan>
+          <range>
+            <min>${min_range}</min>
+            <max>${max_range}</max>
+            <resolution>0.01</resolution>
+          </range>
+        </ray>
+        <plugin name="gazebo_ros_${name2}_controller" filename="libhector_gazebo_ros_sonar.so">
+          <gaussianNoise>0.005</gaussianNoise>
+          <topicName>${ros_topic2}</topicName>
           <bodyName>sonar</bodyName>
           <serviceName>sonar_service</serviceName>
-          <frameId>${name}_link</frameId>
+          <frameId>${name2}_link</frameId>
+        </plugin>
+      </sensor>
+    </gazebo>
+  <link name="${name3}_link">
+      <inertial>
+        <mass value="0.001" />
+        <origin xyz="0 0 0" rpy="0 0 0" />
+        <inertia ixx="0.000000017" ixy="0" ixz="0" iyy="0.000000017" iyz="0" izz="0.000000017" />
+      </inertial>
+        <visual>
+          <origin xyz="0 0 ${height_sonar/2}" rpy="0 0 0"/>
+          <geometry>
+            <box size="${width_sonar} ${width_sonar} ${height_sonar}"/>
+          </geometry>
+          <material name="orange"/>
+        </visual>
+      <collision>
+        <origin xyz="0 0 0" rpy="0 0 0" />
+        <geometry>
+          <box size="0.01 0.01 0.01" />
+        </geometry>
+      </collision>
+  </link>
+  <joint name="${name3}_joint" type="fixed">
+    <axis xyz="0 1 0" />
+     <origin xyz=".0 -.25 0.15" rpy="0 -0.6 -1.5"/>
+    <parent link="chassis"/>
+    <child link="${name3}_link"/>
+  </joint>
+    <gazebo reference="${name3}_link">
+      <sensor type="ray" name="${name3}">
+        <always_on>true</always_on>
+        <update_rate>${update_rate}</update_rate>
+        <pose>0 0 0 0 0 0</pose>
+        <visualize>true</visualize>
+        <ray>
+          <scan>
+            <horizontal>
+              <samples>${ray_count}</samples>
+              <resolution>1</resolution>
+              <min_angle>-${field_of_view/2}</min_angle>
+              <max_angle> ${field_of_view/2}</max_angle>
+            </horizontal>
+            <vertical>
+              <samples>${ray_count}</samples>
+              <resolution>1</resolution>
+              <min_angle>-${field_of_view/2}</min_angle>
+              <max_angle> ${field_of_view/2}</max_angle>
+            </vertical>
+          </scan>
+          <range>
+            <min>${min_range}</min>
+            <max>${max_range}</max>
+            <resolution>0.01</resolution>
+          </range>
+        </ray>
+        <plugin name="gazebo_ros_${name3}_controller" filename="libhector_gazebo_ros_sonar.so">
+          <gaussianNoise>0.005</gaussianNoise>
+          <topicName>${ros_topic3}</topicName>
+          <bodyName>sonar</bodyName>
+          <serviceName>sonar_service</serviceName>
+          <frameId>${name3}_link</frameId>
+        </plugin>
+      </sensor>
+    </gazebo>
+  <link name="${name4}_link">
+      <inertial>
+        <mass value="0.001" />
+        <origin xyz="0 0 0" rpy="0 0 0" />
+        <inertia ixx="0.000000017" ixy="0" ixz="0" iyy="0.000000017" iyz="0" izz="0.000000017" />
+      </inertial>
+        <visual>
+          <origin xyz="0 0 ${height_sonar/2}" rpy="0 0 0"/>
+          <geometry>
+            <box size="${width_sonar} ${width_sonar} ${height_sonar}"/>
+          </geometry>
+          <material name="orange"/>
+        </visual>
+      <collision>
+        <origin xyz="0 0 0" rpy="0 0 0" />
+        <geometry>
+          <box size="0.01 0.01 0.01" />
+        </geometry>
+      </collision>
+  </link>
+  <joint name="${name4}_joint" type="fixed">
+    <axis xyz="0 1 0" />
+     <origin xyz="-.25 0 0.15" rpy="0 -0.6 3.0"/>
+    <parent link="chassis"/>
+    <child link="${name4}_link"/>
+  </joint>
+    <gazebo reference="${name4}_link">
+      <sensor type="ray" name="${name4}">
+        <always_on>true</always_on>
+        <update_rate>${update_rate}</update_rate>
+        <pose>0 0 0 0 0 0</pose>
+        <visualize>true</visualize>
+        <ray>
+          <scan>
+            <horizontal>
+              <samples>${ray_count}</samples>
+              <resolution>1</resolution>
+              <min_angle>-${field_of_view/2}</min_angle>
+              <max_angle> ${field_of_view/2}</max_angle>
+            </horizontal>
+            <vertical>
+              <samples>${ray_count}</samples>
+              <resolution>1</resolution>
+              <min_angle>-${field_of_view/2}</min_angle>
+              <max_angle> ${field_of_view/2}</max_angle>
+            </vertical>
+          </scan>
+          <range>
+            <min>${min_range}</min>
+            <max>${max_range}</max>
+            <resolution>0.01</resolution>
+          </range>
+        </ray>
+        <plugin name="gazebo_ros_${name4}_controller" filename="libhector_gazebo_ros_sonar.so">
+          <gaussianNoise>0.005</gaussianNoise>
+          <topicName>${ros_topic4}</topicName>
+          <bodyName>sonar</bodyName>
+          <serviceName>sonar_service</serviceName>
+          <frameId>${name4}_link</frameId>
         </plugin>
       </sensor>

Commit message: Camera stuff

File: src/roguetwo_description/urdf/em_3905.urdf.xacro (robot description, xacro)
@@ -360,10 +360,11 @@
   <xacro:property name="height1" value="0.05" />
   <xacro:property name="width" value="0.05" />
-  <joint name="fixed" type="fixed">
+<!--   <joint name="fixed" type="fixed">
     <parent link="chassis"/>
     <child link="sensor"/>
   </joint>
+ -->
  <!-- Base Link -->
-  <link name="sensor">
+  <!-- <link name="sensor">
     <collision>
       <origin xyz="0 0 ${height1/2}" rpy="0 0 0"/>
@@ -390,5 +391,5 @@
   <joint name="stereo_joint" type="fixed">
     <axis xyz="0 1 0" />
-    <origin xyz=".1 .0 0.1" rpy="0 0 0"/>
+    <origin xyz=".10 .0 0.15" rpy="0 0 0"/>
     <parent link="base_link"/>
     <child link="sensor"/>
@@ -445,5 +446,4 @@
         <cameraInfoTopicName>camera_info</cameraInfoTopicName>
         <frameName>left_camera_optical_frame</frameName>
-        <!--<rightFrameName>right_camera_optical_frame</rightFrameName>-->
         <hackBaseline>0.07</hackBaseline>
         <distortionK1>0.0</distortionK1>
@@ -455,5 +455,6 @@
     </sensor>
   </gazebo>
-<!--   <link name="camera_stereo_left">
+ -->
+  <link name="camera_stereo_left">
     <collision>
       <origin xyz="0 0 0" rpy="0 0 0"/>
@@ -478,5 +479,5 @@
   <joint name="camera_stereo_left_joint" type="fixed">
     <axis xyz="0 1 0" />
-    <origin xyz=".2 .1 0.1" rpy="0 0 0"/>
+    <origin xyz=".20 .0 0.05" rpy="0 0 0"/>
     <parent link="chassis"/>
     <child link="camera_stereo_left"/>
@@ -514,5 +515,5 @@
     </sensor>
   </gazebo>
-  <link name="camera_stereo_right">
+<!--   <link name="camera_stereo_right">
     <collision>
       <origin xyz="0 0 0" rpy="0 0 0"/>
@@ -745,5 +746,5 @@
   <joint name="${name1}_joint" type="fixed">
     <axis xyz="0 1 0" />
-    <origin xyz=".25 0 0.15" rpy="0 -0.7 0"/>
+    <origin xyz=".25 0 0.15" rpy="0 -0.55 0"/>
     <parent link="chassis"/>
     <child link="${name1}_link"/>
@@ -806,5 +807,5 @@
   <joint name="${name2}_joint" type="fixed">
     <axis xyz="0 1 0" />
-    <origin xyz=".0 .25 0.15" rpy="0 -0.60 1.5"/>
+    <origin xyz=".0 .25 0.15" rpy="0 -0.55 1.5"/>
     <parent link="chassis"/>
     <child link="${name2}_link"/>
@@ -868,5 +869,5 @@
   <joint name="${name3}_joint" type="fixed">
     <axis xyz="0 1 0" />
-     <origin xyz=".0 -.25 0.15" rpy="0 -0.6 -1.5"/>
+     <origin xyz=".0 -.25 0.15" rpy="0 -0.55 -1.5"/>
     <parent link="chassis"/>
     <child link="${name3}_link"/>
@@ -930,5 +931,5 @@
   <joint name="${name4}_joint" type="fixed">
     <axis xyz="0 1 0" />
-     <origin xyz="-.25 0 0.15" rpy="0 -0.6 3.0"/>
+     <origin xyz="-.25 0 0.15" rpy="0 -0.55 3.0"/>
     <parent link="chassis"/>
     <child link="${name4}_link"/>

Commit message: SVO Point Cloud to Octomap

File: src/roguetwo_description/urdf/em_3905.urdf.xacro (robot description, xacro)
@@ -515,5 +515,5 @@
     </sensor>
   </gazebo>
-<!--   <link name="camera_stereo_right">
+  <link name="camera_stereo_right">
     <collision>
       <origin xyz="0 0 0" rpy="0 0 0"/>
@@ -538,5 +538,5 @@
   <joint name="camera_stereo_right_joint" type="fixed">
     <axis xyz="0 1 0" />
-    <origin xyz=".2 -.1 0.1" rpy="0 0 0"/>
+    <origin xyz=".2 -.1 0.05" rpy="0 0 0"/>
     <parent link="chassis"/>
     <child link="camera_stereo_right"/>
@@ -574,5 +574,5 @@
     </sensor>
   </gazebo>
-  <link name="camera_steering">
+<!--   <link name="camera_steering">
     <collision>
       <origin xyz="0 0 0" rpy="0 0 0"/>
