Commit message: bruteforce

File: src/roguetwo_description/urdf/em_3905.urdf.xacro (robot description, xacro)
@@ -710,9 +710,11 @@
   <xacro:property name="height_sonar" value="0.05" />
   <xacro:property name="width_sonar" value="0.05" />
+  <xacro:property name="name5" value="sonar5" />
   <xacro:property name="name1" value="sonar1" />
   <xacro:property name="name2" value="sonar2" />
   <xacro:property name="name3" value="sonar3" />
   <xacro:property name="name4" value="sonar4" />
-  <xacro:property name="ros_topic1" value="/sonar_front_distance" />
+  <xacro:property name="ros_topic5" value="/sonar_frontR_distance" />
+  <xacro:property name="ros_topic1" value="/sonar_frontL_distance" />
   <xacro:property name="ros_topic2" value="/sonar_left_distance" />
   <xacro:property name="ros_topic3" value="/sonar_right_distance" />
@@ -721,6 +723,67 @@
   <xacro:property name="min_range" value="0.02" />
   <xacro:property name="max_range" value="4.5" />
-  <xacro:property name="field_of_view" value="1" />
-  <xacro:property name="ray_count" value="2" />
+  <xacro:property name="field_of_view" value="0.0" />
+  <xacro:property name="ray_count" value="1" />
+  <!-- Base Link -->
+  <link name="${name5}_link">
+      <inertial>
+        <mass value="0.001" />
+        <origin xyz="0 0 0" rpy="0 0 0" />
+        <inertia ixx="0.000000017" ixy="0" ixz="0" iyy="0.000000017" iyz="0" izz="0.000000017" />
+      </inertial>
+        <visual>
+          <origin xyz="0 0 ${height_sonar/2}" rpy="0 0 0"/>
+          <geometry>
+            <box size="${width_sonar} ${width_sonar} ${height_sonar}"/>
+          </geometry>
+          <material name="orange"/>
+        </visual>
+      <collision>
+        <origin xyz="0 0 0" rpy="0 0 0" />
+        <geometry>
+          <box size="0.01 0.01 0.01" />
+        </geometry>
+      </collision>
+  </link>
+  <joint name="${name5}_joint" type="fixed">
+    <axis xyz="0 1 0" />
+    <origin xyz=".25 -.15 0.15" rpy="0 0 0"/>
+    <parent link="chassis"/>
+    <child link="${name5}_link"/>
+  </joint>
+    <gazebo reference="${name5}_link">
+      <sensor type="ray" name="${name5}">
+        <always_on>true</always_on>
+        <update_rate>${update_rate}</update_rate>
+        <pose>0 0 0 0 0 0</pose>
+        <visualize>true</visualize>
+        <ray>
+          <scan>
+            <horizontal>
+              <samples>${ray_count}</samples>
+              <resolution>1</resolution>
+              <min_angle>-${field_of_view/2}</min_angle>
+              <max_angle> ${field_of_view/2}</max_angle>
+            </horizontal>
+            <vertical>
+              <samples>${ray_count}</samples>
+              <resolution>1</resolution>
+              <min_angle>-${field_of_view/2}</min_angle>
+              <max_angle> ${field_of_view/2}</max_angle>
+            </vertical>
+          </scan>
+          <range>
+            <min>${min_range}</min>
+            <max>${max_range}</max>
+            <resolution>0.01</resolution>
+          </range>
+        </ray>
+        <plugin name="gazebo_ros_${name5}_controller" filename="libhector_gazebo_ros_sonar.so">
+          <gaussianNoise>0.005</gaussianNoise>
+          <topicName>${ros_topic5}</topicName>
+          <frameId>${name5}_link</frameId>
+        </plugin>
+      </sensor>
+    </gazebo>
   <!-- Base Link -->
   <link name="${name1}_link">
@@ -746,5 +809,5 @@
   <joint name="${name1}_joint" type="fixed">
     <axis xyz="0 1 0" />
-    <origin xyz=".25 0 0.15" rpy="0 -0.55 0"/>
+    <origin xyz=".25 .15 0.15" rpy="0 0 0"/>
     <parent link="chassis"/>
     <child link="${name1}_link"/>
@@ -807,5 +870,5 @@
   <joint name="${name2}_joint" type="fixed">
     <axis xyz="0 1 0" />
-    <origin xyz=".0 .25 0.15" rpy="0 -0.55 1.5"/>
+    <origin xyz=".0 .25 0.15" rpy="0 0 1.3"/>
     <parent link="chassis"/>
     <child link="${name2}_link"/>
@@ -869,5 +932,5 @@
   <joint name="${name3}_joint" type="fixed">
     <axis xyz="0 1 0" />
-     <origin xyz=".0 -.25 0.15" rpy="0 -0.55 -1.5"/>
+     <origin xyz=".0 -.25 0.15" rpy="0 0 -1.3"/>
     <parent link="chassis"/>
     <child link="${name3}_link"/>
@@ -931,5 +994,5 @@
   <joint name="${name4}_joint" type="fixed">
     <axis xyz="0 1 0" />
-     <origin xyz="-.25 0 0.15" rpy="0 -0.55 3.0"/>
+     <origin xyz="-.25 0 0.15" rpy="0 0 3.14"/>
     <parent link="chassis"/>
     <child link="${name4}_link"/>

Commit message: bruteforce

File: src/roguetwo_description/urdf/em_3905.urdf.xacro (robot description, xacro)
@@ -870,5 +870,5 @@
   <joint name="${name2}_joint" type="fixed">
     <axis xyz="0 1 0" />
-    <origin xyz=".0 .25 0.15" rpy="0 0 1.3"/>
+    <origin xyz="-.12 .21 0.15" rpy="0 0 0.7"/>
     <parent link="chassis"/>
     <child link="${name2}_link"/>
@@ -932,5 +932,5 @@
   <joint name="${name3}_joint" type="fixed">
     <axis xyz="0 1 0" />
-     <origin xyz=".0 -.25 0.15" rpy="0 0 -1.3"/>
+     <origin xyz="-.12 -.21 0.15" rpy="0 0 -0.8"/>
     <parent link="chassis"/>
     <child link="${name3}_link"/>

Commit message: encoder outlier removal, odometry into control & planning, lidar ros ndoe

File: src/roguetwo_description/urdf/em_3905.urdf.xacro (robot description, xacro)
@@ -456,182 +456,4 @@
   </gazebo>
  -->
-  <link name="camera_stereo_left">
-    <collision>
-      <origin xyz="0 0 0" rpy="0 0 0"/>
-      <geometry>
-        <box size="${cameraSize} ${cameraSize} ${cameraSize}"/>
-      </geometry>
-    </collision>
-    <visual>
-      <origin xyz="0 0 0" rpy="0 0 0"/>
-      <geometry>
-        <box size="${cameraSize} ${cameraSize} ${cameraSize}"/>
-      </geometry>
-      <material name="green"/>
-    </visual>
-    <inertial>
-      <mass value="${cameraMass}" />
-      <origin xyz="0 0 0" rpy="0 0 0"/>
-      <box_inertia m="${cameraMass}" x="${cameraSize}" y="${cameraSize}" z="${cameraSize}" />
-      <inertia ixx="1e-6" ixy="0" ixz="0" iyy="1e-6" iyz="0" izz="1e-6" />
-    </inertial>
-  </link>
-  <joint name="camera_stereo_left_joint" type="fixed">
-    <axis xyz="0 1 0" />
-    <origin xyz=".20 .0 0.05" rpy="0 0 0"/>
-    <parent link="chassis"/>
-    <child link="camera_stereo_left"/>
-  </joint>
-  <gazebo reference="camera_stereo_left">
-    <material>Gazebo/Green</material>
-    <sensor type="camera" name="camera_stereo_left">
-      <update_rate>30.0</update_rate>
-      <camera name="head">
-        <horizontal_fov>1.3962634</horizontal_fov>
-        <image>
-          <width>640</width>
-          <height>480</height>
-          <format>R8G8B8</format>
-        </image>
-        <clip>
-          <near>0.02</near>
-          <far>300</far>
-        </clip>
-      </camera>
-      <plugin name="camera_controller" filename="libgazebo_ros_camera.so">
-        <alwaysOn>true</alwaysOn>
-        <updateRate>0.0</updateRate>
-        <cameraName>rogue_two/camera_stereo_left</cameraName>
-        <imageTopicName>image_raw</imageTopicName>
-        <cameraInfoTopicName>camera_info</cameraInfoTopicName>
-        <frameName>camera</frameName>
-        <hackBaseline>0.07</hackBaseline>
-        <distortionK1>0.0</distortionK1>
-        <distortionK2>0.0</distortionK2>
-        <distortionK3>0.0</distortionK3>
-        <distortionT1>0.0</distortionT1>
-        <distortionT2>0.0</distortionT2>
-      </plugin>
-    </sensor>
-  </gazebo>
-  <link name="camera_stereo_right">
-    <collision>
-      <origin xyz="0 0 0" rpy="0 0 0"/>
-      <geometry>
-        <box size="${cameraSize} ${cameraSize} ${cameraSize}"/>
-      </geometry>
-    </collision>
-    <visual>
-      <origin xyz="0 0 0" rpy="0 0 0"/>
-      <geometry>
-        <box size="${cameraSize} ${cameraSize} ${cameraSize}"/>
-      </geometry>
-      <material name="green"/>
-    </visual>
-    <inertial>
-      <mass value="${cameraMass}" />
-      <origin xyz="0 0 0" rpy="0 0 0"/>
-      <box_inertia m="${cameraMass}" x="${cameraSize}" y="${cameraSize}" z="${cameraSize}" />
-      <inertia ixx="1e-6" ixy="0" ixz="0" iyy="1e-6" iyz="0" izz="1e-6" />
-    </inertial>
-  </link>
-  <joint name="camera_stereo_right_joint" type="fixed">
-    <axis xyz="0 1 0" />
-    <origin xyz=".2 -.1 0.05" rpy="0 0 0"/>
-    <parent link="chassis"/>
-    <child link="camera_stereo_right"/>
-  </joint>
-  <gazebo reference="camera_stereo_right">
-    <material>Gazebo/Green</material>
-    <sensor type="camera" name="camera_stereo_right">
-      <update_rate>30.0</update_rate>
-      <camera name="head">
-        <horizontal_fov>1.3962634</horizontal_fov>
-        <image>
-          <width>640</width>
-          <height>480</height>
-          <format>R8G8B8</format>
-        </image>
-        <clip>
-          <near>0.02</near>
-          <far>300</far>
-        </clip>
-      </camera>
-      <plugin name="camera_controller" filename="libgazebo_ros_camera.so">
-        <alwaysOn>true</alwaysOn>
-        <updateRate>0.0</updateRate>
-        <cameraName>rogue_two/camera_stereo_right</cameraName>
-        <imageTopicName>image_raw</imageTopicName>
-        <cameraInfoTopicName>camera_info</cameraInfoTopicName>
-        <frameName>camera</frameName>
-        <hackBaseline>0.07</hackBaseline>
-        <distortionK1>0.0</distortionK1>
-        <distortionK2>0.0</distortionK2>
-        <distortionK3>0.0</distortionK3>
-        <distortionT1>0.0</distortionT1>
-        <distortionT2>0.0</distortionT2>
-      </plugin>
-    </sensor>
-  </gazebo>
-<!--   <link name="camera_steering">
-    <collision>
-      <origin xyz="0 0 0" rpy="0 0 0"/>
-      <geometry>
-        <box size="${cameraSize} ${cameraSize} ${cameraSize}"/>
-      </geometry>
-    </collision>
-    <visual>
-      <origin xyz="0 0 0" rpy="0 0 0"/>
-      <geometry>
-        <box size="${cameraSize} ${cameraSize} ${cameraSize}"/>
-      </geometry>
-      <material name="green"/>
-    </visual>
-    <inertial>
-      <mass value="${cameraMass}" />
-      <origin xyz="0 0 0" rpy="0 0 0"/>
-      <box_inertia m="${cameraMass}" x="${cameraSize}" y="${cameraSize}" z="${cameraSize}" />
-      <inertia ixx="1e-6" ixy="0" ixz="0" iyy="1e-6" iyz="0" izz="1e-6" />
-    </inertial>
-  </link>
-  <joint name="camera_steering_joint" type="fixed">
-    <axis xyz="0 1 0" />
-    <origin xyz=".2 0 0.1" rpy="0 0 0"/>
-    <parent link="chassis"/>
-    <child link="camera_steering"/>
-  </joint>
-  <gazebo reference="camera_steering">
-    <material>Gazebo/Green</material>
-    <sensor type="camera" name="camera_steering">
-      <update_rate>30.0</update_rate>
-      <camera name="head">
-        <horizontal_fov>1.3962634</horizontal_fov>
-        <image>
-          <width>640</width>
-          <height>480</height>
-          <format>R8G8B8</format>
-        </image>
-        <clip>
-          <near>0.02</near>
-          <far>300</far>
-        </clip>
-      </camera>
-      <plugin name="camera_controller" filename="libgazebo_ros_camera.so">
-        <alwaysOn>true</alwaysOn>
-        <updateRate>0.0</updateRate>
-        <cameraName>rogue_two/camera_steering</cameraName>
-        <imageTopicName>image_raw</imageTopicName>
-        <cameraInfoTopicName>camera_info</cameraInfoTopicName>
-        <frameName>camera</frameName>
-        <hackBaseline>0.07</hackBaseline>
-        <distortionK1>0.0</distortionK1>
-        <distortionK2>0.0</distortionK2>
-        <distortionK3>0.0</distortionK3>
-        <distortionT1>0.0</distortionT1>
-        <distortionT2>0.0</distortionT2>
-      </plugin>
-    </sensor>
-  </gazebo>
- -->
 <!--   <xacro:property name="height1" value="0.2" />
   <xacro:property name="width" value="0.2" /> -->
@@ -708,11 +530,13 @@
     <child link="imu"/>
   </joint>
-  <xacro:property name="height_sonar" value="0.05" />
+ <xacro:property name="height_sonar" value="0.05" />
   <xacro:property name="width_sonar" value="0.05" />
+  <xacro:property name="name5" value="sonar5" />
   <xacro:property name="name1" value="sonar1" />
   <xacro:property name="name2" value="sonar2" />
   <xacro:property name="name3" value="sonar3" />
   <xacro:property name="name4" value="sonar4" />
-  <xacro:property name="ros_topic1" value="/sonar_front_distance" />
+  <xacro:property name="ros_topic5" value="/sonar_frontR_distance" />
+  <xacro:property name="ros_topic1" value="/sonar_frontL_distance" />
   <xacro:property name="ros_topic2" value="/sonar_left_distance" />
   <xacro:property name="ros_topic3" value="/sonar_right_distance" />
@@ -721,8 +545,8 @@
   <xacro:property name="min_range" value="0.02" />
   <xacro:property name="max_range" value="4.5" />
-  <xacro:property name="field_of_view" value="1" />
-  <xacro:property name="ray_count" value="2" />
+  <xacro:property name="field_of_view" value="0.0" />
+  <xacro:property name="ray_count" value="1" />
   <!-- Base Link -->
-  <link name="${name1}_link">
+  <link name="${name5}_link">
       <inertial>
         <mass value="0.001" />
@@ -744,7 +568,68 @@
       </collision>
   </link>
+  <joint name="${name5}_joint" type="fixed">
+    <axis xyz="0 1 0" />
+    <origin xyz=".25 -.15 0.15" rpy="0 0 0"/>
+    <parent link="chassis"/>
+    <child link="${name5}_link"/>
+  </joint>
+    <gazebo reference="${name5}_link">
+      <sensor type="ray" name="${name5}">
+        <always_on>true</always_on>
+        <update_rate>${update_rate}</update_rate>
+        <pose>0 0 0 0 0 0</pose>
+        <visualize>true</visualize>
+        <ray>
+          <scan>
+            <horizontal>
+              <samples>${ray_count}</samples>
+              <resolution>1</resolution>
+              <min_angle>-${field_of_view/2}</min_angle>
+              <max_angle> ${field_of_view/2}</max_angle>
+            </horizontal>
+            <vertical>
+              <samples>${ray_count}</samples>
+              <resolution>1</resolution>
+              <min_angle>-${field_of_view/2}</min_angle>
+              <max_angle> ${field_of_view/2}</max_angle>
+            </vertical>
+          </scan>
+          <range>
+            <min>${min_range}</min>
+            <max>${max_range}</max>
+            <resolution>0.01</resolution>
+          </range>
+        </ray>
+        <plugin name="gazebo_ros_${name5}_controller" filename="libhector_gazebo_ros_sonar.so">
+          <gaussianNoise>0.005</gaussianNoise>
+          <topicName>${ros_topic5}</topicName>
+          <frameId>${name5}_link</frameId>
+        </plugin>
+      </sensor>
+    </gazebo>
+  <!-- Base Link -->
+  <link name="${name1}_link">
+      <inertial>
+        <mass value="0.001" />
+        <origin xyz="0 0 0" rpy="0 0 0" />
+        <inertia ixx="0.000000017" ixy="0" ixz="0" iyy="0.000000017" iyz="0" izz="0.000000017" />
+      </inertial>
+        <visual>
+          <origin xyz="0 0 ${height_sonar/2}" rpy="0 0 0"/>
+          <geometry>
+            <box size="${width_sonar} ${width_sonar} ${height_sonar}"/>
+          </geometry>
+          <material name="orange"/>
+        </visual>
+      <collision>
+        <origin xyz="0 0 0" rpy="0 0 0" />
+        <geometry>
+          <box size="0.01 0.01 0.01" />
+        </geometry>
+      </collision>
+  </link>
   <joint name="${name1}_joint" type="fixed">
     <axis xyz="0 1 0" />
-    <origin xyz=".25 0 0.15" rpy="0 -0.55 0"/>
+    <origin xyz=".25 .15 0.15" rpy="0 0 0"/>
     <parent link="chassis"/>
     <child link="${name1}_link"/>
@@ -807,5 +692,5 @@
   <joint name="${name2}_joint" type="fixed">
     <axis xyz="0 1 0" />
-    <origin xyz=".0 .25 0.15" rpy="0 -0.55 1.5"/>
+    <origin xyz="-.12 .21 0.15" rpy="0 0 0.7"/>
     <parent link="chassis"/>
     <child link="${name2}_link"/>
@@ -869,5 +754,5 @@
   <joint name="${name3}_joint" type="fixed">
     <axis xyz="0 1 0" />
-     <origin xyz=".0 -.25 0.15" rpy="0 -0.55 -1.5"/>
+     <origin xyz="-.12 -.21 0.15" rpy="0 0 -0.8"/>
     <parent link="chassis"/>
     <child link="${name3}_link"/>
@@ -931,5 +816,5 @@
   <joint name="${name4}_joint" type="fixed">
     <axis xyz="0 1 0" />
-     <origin xyz="-.25 0 0.15" rpy="0 -0.55 3.0"/>
+     <origin xyz="-.25 0 0.15" rpy="0 0 3.14"/>
     <parent link="chassis"/>
     <child link="${name4}_link"/>

Commit message: bruteforce

File: src/roguetwo_description/urdf/em_3905.urdf.xacro (robot description, xacro)
@@ -870,5 +870,5 @@
   <joint name="${name2}_joint" type="fixed">
     <axis xyz="0 1 0" />
-    <origin xyz="-.12 .21 0.15" rpy="0 0 0.7"/>
+    <origin xyz="-.12 .21 0.15" rpy="0 0 0.76"/>
     <parent link="chassis"/>
     <child link="${name2}_link"/>
@@ -932,5 +932,5 @@
   <joint name="${name3}_joint" type="fixed">
     <axis xyz="0 1 0" />
-     <origin xyz="-.12 -.21 0.15" rpy="0 0 -0.8"/>
+     <origin xyz="-.12 -.21 0.15" rpy="0 0 -0.76"/>
     <parent link="chassis"/>
     <child link="${name3}_link"/>

Commit message: Lidar Mapping working

File: src/roguetwo_description/urdf/em_3905.urdf.xacro (robot description, xacro)
@@ -692,5 +692,5 @@
   <joint name="${name2}_joint" type="fixed">
     <axis xyz="0 1 0" />
-    <origin xyz="-.12 .21 0.15" rpy="0 0 0.7"/>
+    <origin xyz="-.12 .21 0.15" rpy="0 0 0.349"/>
     <parent link="chassis"/>
     <child link="${name2}_link"/>
@@ -754,5 +754,5 @@
   <joint name="${name3}_joint" type="fixed">
     <axis xyz="0 1 0" />
-     <origin xyz="-.12 -.21 0.15" rpy="0 0 -0.8"/>
+     <origin xyz="-.12 -.21 0.15" rpy="0 0 -0.349"/>
     <parent link="chassis"/>
     <child link="${name3}_link"/>
